Commit message: multi_operation

File: clover_description/urdf/camera_sensor.urdf.xacro (robot description, xacro)
@@ -64,5 +64,5 @@
       rate="${rate}"
       horizontal_fov="${horizontal_fov}"
-      frame_name="/${name}_optical"
+      frame_name="${name}_optical"
       k1="${k1}"
       k2="${k2}"

File: clover_description/urdf/clover/clover4.xacro (robot description, xacro)
@@ -7,4 +7,7 @@
   <xacro:arg name="maintain_camera_rate" default="false"/>
   <xacro:arg name="use_clover_physics" default="false"/>
+  <xacro:arg name="mavlink_tcp_port" default="4560"/>
+  <xacro:arg name="sdk_udp_port" default="14540"/>
+  <xacro:arg name="frame_prefix" default=""/>
   <xacro:include filename="clover4_base.xacro" />
   <xacro:include filename="../sensors/rpi_cam.urdf.xacro"/>

File: clover_description/urdf/clover/clover4_gazebo.xacro (robot description, xacro)
@@ -3,5 +3,5 @@
 <robot xmlns:xacro="http://ros.org/wiki/xacro">
   <!-- IMU link -->
-  <link name="/imu_link">
+  <link name="imu_link">
     <inertial>
       <inertia ixx="0.00001" ixy="0.0" ixz="0.0" iyy="0.00001" iyz="0.0" izz="0.00001"/>
@@ -15,5 +15,5 @@
     <origin rpy="0 0 0" xyz="0 0 0"/>
     <parent link="base_link"/>
-    <child link="/imu_link"/>
+    <child link="imu_link"/>
     <!-- <limit upper="0" lower="0" effort="0" velocity="0" /> -->
   </joint>
@@ -46,5 +46,5 @@
       <baroSubTopic>/baro</baroSubTopic>
       <mavlink_addr>INADDR_ANY</mavlink_addr>
-      <mavlink_tcp_port>4560</mavlink_tcp_port>
+      <mavlink_tcp_port>$(arg mavlink_tcp_port)</mavlink_tcp_port>
       <mavlink_udp_port>14560</mavlink_udp_port>
       <serialEnabled>false</serialEnabled>
@@ -54,5 +54,5 @@
       <qgc_udp_port>14550</qgc_udp_port>
       <sdk_addr>INADDR_ANY</sdk_addr>
-      <sdk_udp_port>14540</sdk_udp_port>
+      <sdk_udp_port>$(arg sdk_udp_port)</sdk_udp_port>
       <hil_mode>false</hil_mode>
       <hil_state_level>0</hil_state_level>
@@ -162,5 +162,5 @@
     <plugin name='rotors_gazebo_imu_plugin' filename='libgazebo_imu_plugin.so'>
       <robotNamespace/>
-      <linkName>/imu_link</linkName>
+      <linkName>imu_link</linkName>
       <imuTopic>/imu</imuTopic>
       <gyroscopeNoiseDensity>0.00018665</gyroscopeNoiseDensity>

File: clover_description/urdf/sensors/rpi_cam.urdf.xacro (robot description, xacro)
@@ -2,5 +2,5 @@
 <robot name="rpi_camera" xmlns:xacro="http://ros.org/wiki/xacro">
   <xacro:include filename="../camera_sensor.urdf.xacro"/>
-  <xacro:macro name="rpi_cam" params="name:=rpi_cam parent x:=0 y:=0 z:=0 roll:=0 pitch:=0 yaw:=0 width:=320 height:=240 rate:=40 do_throttling:=false">
+  <xacro:macro name="rpi_cam" params="name:=rpi_cam parent x:=0 y:=0 z:=0 roll:=0 pitch:=0 yaw:=0 width:=1280 height:=960 rate:=40 do_throttling:=false">
     <joint name="${name}_joint" type="fixed">
       <origin xyz="${x} ${y} ${z}"
